File: HeartRateMonitor.kicad_pcb (KiCad board)
At the start: 2 copper layers, 30 x 46.5 mm, 60 parts, among them J1 USB_C_Receptacle_USB2.0, J2 SWD, J3 Conn_01x08_Pin, U1 CH340E, U11 LM2904, U2 LM2904, U3 TLV62130, U4 STM32G030F6Px, U5 TPS60403, U6 LM2904, U9 AD5272BCP

Commit message: add silk
Other:
- board text added: "Yao Haizhou Li bohan Wang Xinshu"
